Commit message: Remove empty links

File: test/pr2.urdf (robot description, URDF)
Before this commit: robot pr2, 95 links, 94 joints
Links:
- removed link head_mount_kinect_ir_optical_frame
- removed link head_mount_kinect_rgb_optical_frame
- removed link head_mount_prosilica_optical_frame
- removed link l_forearm_cam_optical_frame
- removed link l_gripper_l_finger_tip_frame
- removed link l_gripper_led_frame
- removed link l_gripper_tool_frame
- removed link narrow_stereo_l_stereo_camera_optical_frame
- removed link narrow_stereo_optical_frame
- removed link narrow_stereo_r_stereo_camera_optical_frame
- removed link r_forearm_cam_optical_frame
- removed link r_gripper_l_finger_tip_frame
- removed link r_gripper_led_frame
- removed link r_gripper_tool_frame
- removed link wide_stereo_l_stereo_camera_optical_frame
- removed link wide_stereo_optical_frame
- removed link wide_stereo_r_stereo_camera_optical_frame
Joints:
- removed joint head_mount_kinect_ir_optical_frame_joint
- removed joint head_mount_kinect_rgb_optical_frame_joint
- removed joint head_mount_prosilica_optical_frame_joint
- removed joint l_forearm_cam_optical_frame_joint
- removed joint l_gripper_joint
- removed joint l_gripper_led_joint
- removed joint l_gripper_tool_joint
- removed joint narrow_stereo_l_stereo_camera_optical_frame_joint
- removed joint narrow_stereo_optical_frame_joint
- removed joint narrow_stereo_r_stereo_camera_optical_frame_joint
- removed joint r_forearm_cam_optical_frame_joint
- removed joint r_gripper_joint
- removed joint r_gripper_led_joint
- removed joint r_gripper_tool_joint
- removed joint wide_stereo_l_stereo_camera_optical_frame_joint
- removed joint wide_stereo_optical_frame_joint
- removed joint wide_stereo_r_stereo_camera_optical_frame_joint
